File: hardware/tinymac.brd (EAGLE design)
At the start: 43 x 41.4 mm, 29 parts, among them IC1 LPC1114FN28, J1 ZX62-B-5PA, SW1 TACT_SW, SW2 TACT_SW, SW3 TACT_SW, SW4 TACT_SW, SW5 TACT_SW, T1 TA48M033F

Commit message: edit board net
Routing:
- net +3.3V: track 57.7 -> 81.2 mm
- net +3.3V_TGT: track 18.9 -> 4.46 mm
- net N$19: track 0.00 -> 6.15 mm
- net GND: track 139.7 -> 142.1 mm
- net N$2: track 19.9 -> 18.6 mm
Changed lines of the file:
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@@
 <wire x1="17.6022" y1="25.3746" x2="17.78" y2="25.4" width="0.254" layer="1"/>
 <wire x1="17.6022" y1="22.1742" x2="17.5" y2="22.14" width="0.254" layer="1"/>
-<wire x1="25.146" y1="20.8026" x2="25.146" y2="14.6304" width="0.254" layer="1"/>
-<wire x1="25.146" y1="14.6304" x2="25.12" y2="14.52" width="0.254" layer="1"/>
-<wire x1="25.146" y1="20.8026" x2="25.02" y2="21.02" width="0.254" layer="1"/>
-<wire x1="23.5458" y1="22.4028" x2="17.6022" y2="22.4028" width="0.254" layer="1"/>
-<wire x1="24.9174" y1="21.0312" x2="23.5458" y2="22.4028" width="0.254" layer="1"/>
+<wire x1="22.1742" y1="21.0312" x2="24.9174" y2="21.0312" width="0.254" layer="1"/>
+<wire x1="20.8026" y1="22.4028" x2="22.1742" y2="21.0312" width="0.254" layer="1"/>
+<wire x1="17.6022" y1="22.4028" x2="20.8026" y2="22.4028" width="0.254" layer="1"/>
+<wire x1="24.9174" y1="21.0312" x2="25.02" y2="21.02" width="0.254" layer="1"/>
 <wire x1="17.6022" y1="22.4028" x2="17.5" y2="22.14" width="0.254" layer="1"/>
-<wire x1="24.9174" y1="21.0312" x2="25.02" y2="21.02" width="0.254" layer="1"/>
 <wire x1="9.8298" y1="20.8026" x2="9.8298" y2="14.6304" width="0.254" layer="16"/>
 <wire x1="9.8298" y1="14.6304" x2="9.88" y2="14.52" width="0.254" layer="16"/>
@@
 <wire x1="17.6022" y1="7.0866" x2="17.5" y2="6.9" width="0.254" layer="16"/>
 <wire x1="20.1168" y1="10.0584" x2="20.32" y2="10.16" width="0.254" layer="16"/>
+<wire x1="23.7744" y1="14.4018" x2="24.9174" y2="14.4018" width="0.254" layer="1"/>
+<wire x1="20.1168" y1="10.7442" x2="23.7744" y2="14.4018" width="0.254" layer="1"/>
+<wire x1="24.9174" y1="14.4018" x2="25.12" y2="14.52" width="0.254" layer="1"/>
+<wire x1="20.1168" y1="10.7442" x2="20.32" y2="10.16" width="0.254" layer="1"/>
 <wire x1="23.5458" y1="6.858" x2="25.4" y2="6.858" width="0.254" layer="16"/>
 <wire x1="20.3454" y1="10.0584" x2="23.5458" y2="6.858" width="0.254" layer="16"/>
@@
 <wire x1="10.0584" y1="14.6304" x2="9.88" y2="14.52" width="0.254" layer="16"/>
 <wire x1="17.3736" y1="13.4874" x2="17.4" y2="13.4" width="0.254" layer="16"/>
-<wire x1="23.7744" y1="14.4018" x2="24.9174" y2="14.4018" width="0.254" layer="1"/>
-<wire x1="20.1168" y1="10.7442" x2="23.7744" y2="14.4018" width="0.254" layer="1"/>
-<wire x1="24.9174" y1="14.4018" x2="25.12" y2="14.52" width="0.254" layer="1"/>
-<wire x1="20.1168" y1="10.7442" x2="20.32" y2="10.16" width="0.254" layer="1"/>
+<wire x1="17.6022" y1="13.4874" x2="17.6022" y2="21.9456" width="0.254" layer="1"/>
+<wire x1="17.6022" y1="21.9456" x2="17.5" y2="22.14" width="0.254" layer="1"/>
+<wire x1="17.6022" y1="13.4874" x2="17.4" y2="13.4" width="0.254" layer="1"/>
 <wire x1="13.9446" y1="34.29" x2="12.66" y2="34.29" width="0.254" layer="1"/>
 <wire x1="17.6022" y1="30.6324" x2="14.6304" y2="33.6042" width="0.254" layer="1"/>
@@
 <contactref element="VCC" pad="1"/>
 <contactref element="R6" pad="2"/>
+<contactref element="R1" pad="2"/>
 <wire x1="20.8026" y1="25.6032" x2="20.3454" y2="25.6032" width="0.254" layer="16"/>
 <wire x1="24.003" y1="28.8036" x2="20.8026" y2="25.6032" width="0.254" layer="16"/>
 <wire x1="27.8892" y1="28.8036" x2="24.003" y2="28.8036" width="0.254" layer="16"/>
-<wire x1="29.0322" y1="29.9466" x2="28.575" y2="29.4894" width="0.254" layer="16"/>
-<wire x1="28.575" y1="29.4894" x2="27.8892" y2="28.8036" width="0.254" layer="16"/>
+<wire x1="29.0322" y1="29.9466" x2="27.8892" y2="28.8036" width="0.254" layer="16"/>
 <wire x1="29.0322" y1="31.0896" x2="29.0322" y2="29.9466" width="0.254" layer="16"/>
 <wire x1="28.3464" y1="31.7754" x2="29.0322" y2="31.0896" width="0.254" layer="16"/>
@@
 <wire x1="28.3464" y1="31.7754" x2="29.9466" y2="33.3756" width="0.254" layer="16"/>
 <wire x1="29.9466" y1="36.576" x2="30" y2="36.64" width="0.254" layer="16"/>
-<wire x1="31.5468" y1="26.5176" x2="28.575" y2="29.4894" width="0.254" layer="16"/>
-<wire x1="31.5468" y1="3.6576" x2="31.5468" y2="26.5176" width="0.254" layer="16"/>
-<wire x1="30.6324" y1="2.7432" x2="31.5468" y2="3.6576" width="0.254" layer="16"/>
-<wire x1="30.6324" y1="2.7432" x2="30.48" y2="2.54" width="0.254" layer="16"/>
-<contactref element="R1" pad="2"/>
-<wire x1="31.5468" y1="3.6576" x2="30.48" y2="14.605" width="0" layer="19" extent="16-16"/>
-<wire x1="7.62" y1="2.54" x2="30.48" y2="2.54" width="0" layer="19" extent="1-1"/>
+<wire x1="10.9728" y1="2.5146" x2="7.7724" y2="2.5146" width="0.254" layer="1"/>
+<wire x1="12.1158" y1="1.3716" x2="10.9728" y2="2.5146" width="0.254" layer="1"/>
+<wire x1="29.2608" y1="1.3716" x2="12.1158" y2="1.3716" width="0.254" layer="1"/>
+<wire x1="30.4038" y1="2.5146" x2="29.2608" y2="1.3716" width="0.254" layer="1"/>
+<wire x1="7.7724" y1="2.5146" x2="7.62" y2="2.54" width="0.254" layer="1"/>
+<wire x1="30.4038" y1="2.5146" x2="30.48" y2="2.54" width="0.254" layer="1"/>
+<wire x1="30.6324" y1="12.1158" x2="30.6324" y2="14.4018" width="0.254" layer="1"/>
+<wire x1="31.5468" y1="11.2014" x2="30.6324" y2="12.1158" width="0.254" layer="1"/>
+<wire x1="31.5468" y1="3.6576" x2="31.5468" y2="11.2014" width="0.254" layer="1"/>
+<wire x1="30.6324" y1="2.7432" x2="31.5468" y2="3.6576" width="0.254" layer="1"/>
+<wire x1="30.6324" y1="14.4018" x2="30.48" y2="14.605" width="0.254" layer="1"/>
+<wire x1="30.6324" y1="2.7432" x2="30.48" y2="2.54" width="0.254" layer="1"/>
+<wire x1="27.8892" y1="27.6606" x2="27.8892" y2="28.8036" width="0.254" layer="16"/>
+<wire x1="29.4894" y1="26.0604" x2="27.8892" y2="27.6606" width="0.254" layer="16"/>
+<wire x1="29.4894" y1="15.5448" x2="29.4894" y2="26.0604" width="0.254" layer="16"/>
+<wire x1="30.4038" y1="14.6304" x2="29.4894" y2="15.5448" width="0.254" layer="16"/>
+<wire x1="30.4038" y1="14.6304" x2="30.48" y2="14.605" width="0.254" layer="16"/>
 </signal>
 <signal name="VBUS">
@@
 <wire x1="30.4038" y1="20.8026" x2="30.48" y2="20.955" width="0.254" layer="1"/>
 <wire x1="30.6324" y1="21.0312" x2="30.48" y2="20.955" width="0.254" layer="1"/>
-<wire x1="20.3454" y1="20.8026" x2="20.3454" y2="14.6304" width="0.254" layer="1"/>
+<wire x1="20.3454" y1="20.8026" x2="20.3454" y2="17.8308" width="0.254" layer="1"/>
+<wire x1="20.3454" y1="17.8308" x2="20.3454" y2="14.6304" width="0.254" layer="1"/>
 <wire x1="20.3454" y1="14.6304" x2="20.42" y2="14.52" width="0.254" layer="1"/>
 <wire x1="20.3454" y1="20.8026" x2="20.42" y2="21.02" width="0.254" layer="1"/>
-<wire x1="24.003" y1="17.6022" x2="27.8892" y2="17.6022" width="0.254" layer="16"/>
-<wire x1="21.0312" y1="14.6304" x2="24.003" y2="17.6022" width="0.254" layer="16"/>
-<wire x1="20.574" y1="14.6304" x2="21.0312" y2="14.6304" width="0.254" layer="16"/>
-<wire x1="27.8892" y1="17.6022" x2="27.94" y2="17.78" width="0.254" layer="16"/>
-<wire x1="20.574" y1="14.6304" x2="20.42" y2="14.52" width="0.254" layer="16"/>
+<wire x1="20.3454" y1="17.8308" x2="27.8892" y2="17.8308" width="0.254" layer="1"/>
+<wire x1="27.8892" y1="17.8308" x2="27.94" y2="17.78" width="0.254" layer="1"/>
 </signal>
 <signal name="N$6">
@@
 <contactref element="LED" pad="1"/>
 <contactref element="R6" pad="1"/>
-<wire x1="7.62" y1="5.08" x2="12.7" y2="2.54" width="0" layer="19" extent="1-1"/>
+<wire x1="10.287" y1="5.0292" x2="7.7724" y2="5.0292" width="0.254" layer="1"/>
+<wire x1="12.573" y1="2.7432" x2="10.287" y2="5.0292" width="0.254" layer="1"/>
+<wire x1="7.7724" y1="5.0292" x2="7.62" y2="5.08" width="0.254" layer="1"/>
+<wire x1="12.573" y1="2.7432" x2="12.7" y2="2.54" width="0.254" layer="1"/>
 </signal>
 <signal name="N$9">
@@
 <wire x1="17.8308" y1="10.0584" x2="17.78" y2="10.16" width="0.254" layer="1"/>
 <wire x1="20.1168" y1="6.858" x2="20.32" y2="6.858" width="0.254" layer="1"/>
-<wire x1="29.2608" y1="14.4018" x2="30.4038" y2="14.4018" width="0.254" layer="16"/>
-<wire x1="26.7462" y1="11.8872" x2="29.2608" y2="14.4018" width="0.254" layer="16"/>
-<wire x1="19.431" y1="11.8872" x2="26.7462" y2="11.8872" width="0.254" layer="16"/>
-<wire x1="17.8308" y1="10.287" x2="19.431" y2="11.8872" width="0.254" layer="16"/>
-<wire x1="17.8308" y1="10.287" x2="17.78" y2="10.16" width="0.254" layer="16"/>
 </signal>
 <signal name="N$1">

Commit message: try full GND
Routing:
- net GND: track 142.1 -> 0.00 mm
- net +3.3V: track 81.2 -> 125.8 mm
- net N$6: track 25.9 -> 48.3 mm
- net N$4: track 15.8 -> 21.9 mm
- net N$9: track 13.3 -> 16.7 mm
- net N$17: track 17.4 -> 19.3 mm
- net VBUS: track 19.7 -> 19.2 mm, vias 0 -> 1
- added copper zone on layer 1, net GND
