File: hardware/tinymac.brd (EAGLE design)
At the start: 43 x 41.4 mm, 29 parts, among them IC1 LPC1114FN28, J1 ZX62-B-5PA, SW1 TACT_SW, SW2 TACT_SW, SW3 TACT_SW, SW4 TACT_SW, SW5 TACT_SW, T1 TA48M033F

Commit message: apply pin setting in firmware code as schematic
Connections:
- net N$10 renamed RST
- net N$12 renamed SCE
- net N$15 renamed SW_INPUT
- net N$4 renamed MOSI
- net N$5 renamed SCLK
- net N$9 renamed DC
Changed lines of the file:
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@@
 <wire x1="20.2184" y1="39.7256" x2="20.364" y2="39.875" width="0.4064" layer="1"/>
 </signal>
-<signal name="N$15">
+<signal name="SW_INPUT">
 <contactref element="SW1" pad="2-A"/>
 <contactref element="SW1" pad="1-A"/>
@@
 <wire x1="24.9936" y1="11.8872" x2="24.9936" y2="11.7856" width="0.254" layer="1"/>
 </signal>
-<signal name="N$4">
+<signal name="MOSI">
 <contactref element="MOSI" pad="1"/>
 <contactref element="IC1" pad="2"/>
@@
 <wire x1="17.4752" y1="2.54" x2="17.526" y2="2.54" width="0.254" layer="1"/>
 </signal>
-<signal name="N$5">
+<signal name="SCLK">
 <contactref element="IC1" pad="6"/>
 <contactref element="SCLK" pad="1"/>
@@
 <wire x1="12.3952" y1="2.54" x2="12.446" y2="2.54" width="0.4064" layer="1"/>
 </signal>
-<signal name="N$9">
+<signal name="DC">
 <contactref element="DC" pad="1"/>
 <contactref element="IC1" pad="4"/>
@@
 <wire x1="20.0152" y1="2.54" x2="20.066" y2="2.54" width="0.254" layer="1"/>
 </signal>
-<signal name="N$10">
+<signal name="RST">
 <contactref element="RST" pad="1"/>
 <contactref element="IC1" pad="10"/>
@@
 <wire x1="22.6568" y1="2.54" x2="22.606" y2="2.54" width="0.254" layer="1"/>
 </signal>
-<signal name="N$12">
+<signal name="SCE">
 <contactref element="IC1" pad="11"/>
 <contactref element="SCE" pad="1"/>
